File: hardware/controlboard_SMD/pfm3_ctrl.sch (KiCad schematic (older format))
At the start: 55 parts, among them J1 pfm3ControlBoard, J2 Ext, J3 0 ohm, SW1 Push, SW10 Push, SW11 Push, SW12 Push, SW2 Push, SW3 Push, SW4 Push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

Commit message: Control board v1.1
Parts:
- Enc1: value Encoder -> a
- Enc2: value Encoder -> b
- Enc3: value Encoder -> c
- Enc4: value Encoder -> d
- Enc5: value Encoder -> e
- Enc6: value Encoder -> f
Other:
- moved on the sheet: Enc2, Enc3, Enc4, Enc5
Changed lines of the file:
@@
 P 10350 2550
 F 0 "Enc1" H 10293 2183 50  0000 C CNN
-F 1 "Encoder" H 10293 2274 50  0000 C CNN
+F 1 "a" H 10293 2274 50  0000 C CNN
 F 2 "A_PFM3:FMEncoder2_pfm3" H 10200 2710 50  0001 C CNN
 F 3 "~" H 10350 2810 50  0001 C CNN
@@
 L Device:Rotary_Encoder Enc3
 U 1 1 5D17414B
+P 10350 3900
+F 0 "Enc3" H 10293 3533 50  0000 C CNN
+F 1 "c" H 10293 3624 50  0000 C CNN
+F 2 "A_PFM3:FMEncoder2_pfm3" H 10200 4060 50  0001 C CNN
+F 3 "~" H 10350 4160 50  0001 C CNN
+	1    10350 3900
+	-1   0    0    1
+$EndComp
+Wire Wire Line
+	10650 3150 11250 3150
+Wire Wire Line
+	10650 3350 11250 3350
+Wire Wire Line
+	10650 3250 10750 3250
+$Comp
+L Device:Rotary_Encoder Enc5
+U 1 1 5D17888E
+P 11700 3250
+F 0 "Enc5" H 11643 2883 50  0000 C CNN
+F 1 "e" H 11643 2974 50  0000 C CNN
+F 2 "A_PFM3:FMEncoder2_pfm3" H 11550 3410 50  0001 C CNN
+F 3 "~" H 11700 3510 50  0001 C CNN
+	1    11700 3250
+	-1   0    0    1
+$EndComp
+Wire Wire Line
+	10650 3800 11250 3800
+Wire Wire Line
+	10650 4000 11250 4000
+Wire Wire Line
+	10650 3900 10750 3900
+$Comp
+L Device:Rotary_Encoder Enc2
+U 1 1 5D17D652
 P 10350 3250
-F 0 "Enc3" H 10293 2883 50  0000 C CNN
-F 1 "Encoder" H 10293 2974 50  0000 C CNN
+F 0 "Enc2" H 10293 2883 50  0000 C CNN
+F 1 "b" H 10293 2974 50  0000 C CNN
 F 2 "A_PFM3:FMEncoder2_pfm3" H 10200 3410 50  0001 C CNN
 F 3 "~" H 10350 3510 50  0001 C CNN
@@
 $EndComp
 Wire Wire Line
-	10650 3150 11250 3150
-Wire Wire Line
-	10650 3350 11250 3350
-Wire Wire Line
-	10650 3250 10750 3250
-$Comp
-L Device:Rotary_Encoder Enc5
-U 1 1 5D17888E
-P 10350 3900
-F 0 "Enc5" H 10293 3533 50  0000 C CNN
-F 1 "Encoder" H 10293 3624 50  0000 C CNN
-F 2 "A_PFM3:FMEncoder2_pfm3" H 10200 4060 50  0001 C CNN
-F 3 "~" H 10350 4160 50  0001 C CNN
-	1    10350 3900
-	-1   0    0    1
-$EndComp
-Wire Wire Line
-	10650 3800 11250 3800
-Wire Wire Line
-	10650 4000 11250 4000
-Wire Wire Line
-	10650 3900 10750 3900
-$Comp
-L Device:Rotary_Encoder Enc2
-U 1 1 5D17D652
+	12000 2450 12600 2450
+Wire Wire Line
+	12000 2650 12600 2650
+Wire Wire Line
+	12000 2550 12100 2550
+$Comp
+L Device:Rotary_Encoder Enc4
+U 1 1 5D18299A
 P 11700 2550
-F 0 "Enc2" H 11643 2183 50  0000 C CNN
-F 1 "Encoder" H 11643 2274 50  0000 C CNN
+F 0 "Enc4" H 11643 2183 50  0000 C CNN
+F 1 "d" H 11643 2274 50  0000 C CNN
 F 2 "A_PFM3:FMEncoder2_pfm3" H 11550 2710 50  0001 C CNN
 F 3 "~" H 11700 2810 50  0001 C CNN
@@
 $EndComp
 Wire Wire Line
-	12000 2450 12600 2450
-Wire Wire Line
-	12000 2650 12600 2650
-Wire Wire Line
-	12000 2550 12100 2550
-$Comp
-L Device:Rotary_Encoder Enc4
-U 1 1 5D18299A
-P 11700 3250
-F 0 "Enc4" H 11643 2883 50  0000 C CNN
-F 1 "Encoder" H 11643 2974 50  0000 C CNN
-F 2 "A_PFM3:FMEncoder2_pfm3" H 11550 3410 50  0001 C CNN
-F 3 "~" H 11700 3510 50  0001 C CNN
-	1    11700 3250
-	-1   0    0    1
-$EndComp
-Wire Wire Line
 	12000 3150 12600 3150
 Wire Wire Line
@@
 P 11700 3900
 F 0 "Enc6" H 11643 3533 50  0000 C CNN
-F 1 "Encoder" H 11643 3624 50  0000 C CNN
+F 1 "f" H 11643 3624 50  0000 C CNN
 F 2 "A_PFM3:FMEncoder2_pfm3" H 11550 4060 50  0001 C CNN
 F 3 "~" H 11700 4160 50  0001 C CNN
@@
 	3500 1800 3500 2250
 $Comp
-L power:GND #PWR?
+L power:GND #PWR0101
 U 1 1 5EF1F56A
 P 7850 10100
-F 0 "#PWR?" H 7850 9850 50  0001 C CNN
+F 0 "#PWR0101" H 7850 9850 50  0001 C CNN
 F 1 "GND" H 7855 9927 50  0000 C CNN
 F 2 "" H 7850 10100 50  0001 C CNN

Commit message: PCB controlboard 1.2 proto
Parts:
- removed Enc1: a, A_PFM3:FMEncoder2_pfm3, symbol Device:Rotary_Encoder
- removed Enc2: b, A_PFM3:FMEncoder2_pfm3, symbol Device:Rotary_Encoder
- removed Enc3: c, A_PFM3:FMEncoder2_pfm3, symbol Device:Rotary_Encoder
- removed Enc4: d, A_PFM3:FMEncoder2_pfm3, symbol Device:Rotary_Encoder
- removed Enc5: e, A_PFM3:FMEncoder2_pfm3, symbol Device:Rotary_Encoder
- removed Enc6: f, A_PFM3:FMEncoder2_pfm3, symbol Device:Rotary_Encoder
- removed J2: Ext, A_PFM3:CtrlBoard_exp_1x08, symbol Connector:Conn_01x08_Female
- removed J3: 0 ohm, Resistor_SMD:R_0402_1005Metric, symbol Connector_Generic:Conn_01x02
- added C4: 100nF, Capacitor_SMD:C_0402_1005Metric, symbol Device:C
- added Enc1: a, A_PFM3:FMEncoder2_pfm3, symbol Device:Rotary_Encoder_Switch
- added Enc2: b, A_PFM3:FMEncoder2_pfm3, symbol Device:Rotary_Encoder_Switch
- added Enc3: c, A_PFM3:FMEncoder2_pfm3, symbol Device:Rotary_Encoder_Switch
- added Enc4: d, A_PFM3:FMEncoder2_pfm3, symbol Device:Rotary_Encoder_Switch
- added Enc5: e, A_PFM3:FMEncoder2_pfm3, symbol Device:Rotary_Encoder_Switch
- added Enc6: f, A_PFM3:FMEncoder2_pfm3, symbol Device:Rotary_Encoder_Switch
- added J2: Ext, Connector_PinSocket_2.54mm:PinSocket_1x10_P2.54mm_Vertical, symbol Connector_Generic:Conn_01x10
- added J4: ExtButton, Connector_PinSocket_2.54mm:PinSocket_1x03_P2.54mm_Vertical, symbol Connector_Generic:Conn_01x03
- added R26, R27, R28, R29, R30, R31, R32, R33: 10k, Resistor_SMD:R_0402_1005Metric, symbol Device:R
- added U4: 74hc165, Package_SO:SOIC-16_3.9x9.9mm_P1.27mm, symbol 74xx_IEEE:74165
Connections:
- net labels added: EncBut1, EncBut2, EncBut3, EncBut4, EncBut5, EncBut6
- wire segments 211 -> 293
Other:
- moved on the sheet: C1, C2, C3, D1, R1, R10, R11, R12, R13, R14, R15, R16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
