File: hardware/3DCasePCB/topsurface_v2.x/pfm3_topsurface.kicad_pcb (KiCad board)
At the start: 2 copper layers, 208 x 95.7 mm, 7 parts, among them J13 TFT / SD

Commit message: v2.0 JLCPCB ordered for test
Other:
- board text added: "(st)"
