File: hardware/controlboard_SMD/v2.x/pfm3_ctrl.kicad_pcb (KiCad board)
At the start: 2 copper layers, 135 x 87 mm, 61 parts, among them J1 pfm3ControlBoard, SW1 Push, SW10 Push, SW11 Push, SW12 Push, SW2 Push, SW3 Push, SW4 Push, SW5 Push, SW6 Push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

Commit message: Small control board PCB modification: wider clearance around placement holes
Other:
- board text added: "preenfm3 control v2.0.1 SMD Xavier Hosxe May 2023"
- board text removed: "preenfm3 control v2.0 SMD Xavier Hosxe 11/2022"
Changed lines of the file:
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@@
       (drillshape 0)
       (scaleselection 1)
-      (outputdirectory "v2.0/gerber_v2.0/"))
+      (outputdirectory "v2.0/cb_gerber_v2.01/"))
   )
   (net 0 "")
@@
     (pad 6 thru_hole circle (at 3.81 55.245) (size 1.524 1.524) (drill 0.762) (layers *.Cu *.Mask)
       (net 37 /LED))
-    (pad "" thru_hole circle (at 0 -0.635) (size 3.5 3.5) (drill 3.5) (layers *.Cu *.Mask))
-    (pad "" thru_hole circle (at 64.77 -25.4) (size 3.5 3.5) (drill 3.5) (layers *.Cu *.Mask))
-    (pad "" thru_hole circle (at -63.881 -0.635) (size 3.5 3.5) (drill 3.5) (layers *.Cu *.Mask))
-    (pad "" thru_hole circle (at 64.77 55.245) (size 3.5 3.5) (drill 3.5) (layers *.Cu *.Mask))
-    (pad "" thru_hole circle (at -63.881 55.245) (size 3.5 3.5) (drill 3.5) (layers *.Cu *.Mask))
+    (pad "" thru_hole circle (at 0 -0.635) (size 3.5 3.5) (drill 3.5) (layers *.Cu *.Mask)
+      (clearance 1))
+    (pad "" thru_hole circle (at 64.77 -25.4) (size 3.5 3.5) (drill 3.5) (layers *.Cu *.Mask)
+      (clearance 1))
+    (pad "" thru_hole circle (at -63.881 -0.635) (size 3.5 3.5) (drill 3.5) (layers *.Cu *.Mask)
+      (clearance 1))
+    (pad "" thru_hole circle (at 64.77 55.245) (size 3.5 3.5) (drill 3.5) (layers *.Cu *.Mask)
+      (clearance 1))
+    (pad "" thru_hole circle (at -63.881 55.245) (size 3.5 3.5) (drill 3.5) (layers *.Cu *.Mask)
+      (clearance 1))
     (pad 5 thru_hole circle (at 1.27 55.245) (size 1.524 1.524) (drill 0.762) (layers *.Cu *.Mask)
       (net 5 /h165_clk))
@@
     (effects (font (size 2 2) (thickness 0.3)))
   )
-  (gr_text "preenfm3 control \nv2.0 SMD\nXavier Hosxe\n11/2022" (at 69.723 39.37) (layer F.SilkS)
+  (gr_text "preenfm3 control \nv2.0.1 SMD\nXavier Hosxe\nMay 2023" (at 69.723 39.37) (layer F.SilkS)
     (effects (font (size 1.5 1.5) (thickness 0.2)) (justify left))
   )
